File: hardware/Autonomous Rover Kicad.kicad_pcb (KiCad board)
At the start: 2 copper layers, 101.6 x 101.6 mm, 6 parts, among them J1 MPU6050, J2 Arducam OV2640, J3 Conn_02x20_Odd_Even, J4 9V Battery Input, J5 L298N Logic, J6 L298N Power

Commit message: Hardware: bring decoupling caps onto the PCB + refresh schematic image
- PCB: C1/C2/C3 placed and routed, copper pour updated. Verified with
  kicad-cli: DRC 0 violations, 0 unconnected items.
- Replace the stale Schematic.png with an up-to-date Schematic.svg that shows
  the net labels, no-connect flags, and the three decoupling caps; README now
  points to the SVG (opaque light background, renders in light and dark themes).
- gitignore KiCad editor lock files.

Co-Authored-By: Claude Opus 4.8 <noreply@anthropic.com>
Parts:
- added C1: 100uF, Capacitor_THT:CP_Radial_D6.3mm_P2.50mm, F.Cu at (155.3, 139.3)
- added C2: 470uF, Capacitor_THT:CP_Radial_D8.0mm_P3.50mm, F.Cu at (155.7, 130.7)
- added C3: 10uF, Capacitor_THT:CP_Radial_D5.0mm_P2.50mm, F.Cu at (162.6, 138.7)
- J3: value Conn_02x20_Odd_Even -> ESP32-S3
- moved J1 42.4 mm to (123.0, 71.9)
- moved J3 42.4 mm to (91.5, 86.4)
- moved J5 42.4 mm to (115.0, 67.4)
- moved J4 42.4 mm to (165.1, 102.5)
- moved J2 42.4 mm to (143.1, 99.3)
- moved J6 42.4 mm to (132.6, 138.2)
Connections:
- net Net-(J1-Pin_3) renamed /I2C_SCL
- net Net-(J1-Pin_4) renamed /I2C_SDA
- net Net-(J2-Pin_5) renamed /CAM_SPI1
- net Net-(J2-Pin_6) renamed /CAM_SPI2
- net Net-(J2-Pin_7) renamed /CAM_SPI4
- net Net-(J2-Pin_8) renamed /CAM_SPI3
- net Net-(J3-Pin_10) renamed /MOT_CTRL5
- net Net-(J3-Pin_12) renamed /MOT_CTRL6
- net Net-(J3-Pin_2) renamed /MOT_CTRL1
- net Net-(J3-Pin_4) renamed /MOT_CTRL2
- net Net-(J3-Pin_6) renamed /MOT_CTRL3
- net Net-(J3-Pin_8) renamed /MOT_CTRL4
Routing:
- net Net-(J1-Pin_1): track 116.7 -> 195.5 mm
- net Net-(J3-Pin_38): track 48.0 -> 117.9 mm
- net GND: track 169.9 -> 212.6 mm
- net Net-(J4-Pin_1): track 49.1 -> 76.9 mm
Other:
- board size 101.6 x 101.6 mm -> 92.3 x 86.2 mm
- board text added: "UCSD ECE Design Competition"
- board text removed: "UCSD ECE Design Competition - Autonomous Rover"
